Commit message: adding meshes

File: resources/obj/random_urdfs/000/000.urdf (robot description, URDF)
Before this commit: robot blob000, 1 links, 0 joints
Links:
- link random_obj_000: geometry collision mesh filename=000_coll.stl scale=0.0076 0.0076 0.0076; visual mesh filename=000.stl scale=0.0076 0.0076 0.0076

File: resources/obj/random_urdfs/001/001.urdf (robot description, URDF)
Before this commit: robot blob001, 1 links, 0 joints
Links:
- link random_obj_001: geometry collision mesh filename=001_coll.stl scale=0.0090 0.0090 0.0090; visual mesh filename=001.stl scale=0.0090 0.0090 0.0090

File: resources/obj/random_urdfs/002/002.urdf (robot description, URDF)
Before this commit: robot blob002, 1 links, 0 joints
Links:
- link random_obj_002: geometry collision mesh filename=002_coll.stl scale=0.0071 0.0071 0.0071; visual mesh filename=002.stl scale=0.0071 0.0071 0.0071

File: resources/obj/random_urdfs/003/003.urdf (robot description, URDF)
Before this commit: robot blob003, 1 links, 0 joints
Links:
- link random_obj_003: geometry collision mesh filename=003_coll.stl scale=0.0064 0.0064 0.0064; visual mesh filename=003.stl scale=0.0064 0.0064 0.0064
